Commit message: simulation_v_1

File: nexus_4wd_mecanum_simulator/nexus_4wd_mecanum_description/urdf/nexus_4wd_mecanum.xacro (robot description, xacro)
@@ -12,5 +12,5 @@
   <link name="base_footprint"></link>
   <joint name="base_link_joint" type="fixed">
-    <origin xyz="0 0 0.05" rpy="0 0 0" />
+    <origin xyz="1 0 0.05" rpy="0 0 0" />
     <parent link="base_footprint"/>
     <child link="base_link" />

Commit message: simulation_v_2

File: nexus_4wd_mecanum_simulator/nexus_4wd_mecanum_description/urdf/nexus_4wd_mecanum.xacro (robot description, xacro)
@@ -12,5 +12,5 @@
   <link name="base_footprint"></link>
   <joint name="base_link_joint" type="fixed">
-    <origin xyz="1 0 0.05" rpy="0 0 0" />
+    <origin xyz="1 -0.18 0.05" rpy="0 0 0" />
     <parent link="base_footprint"/>
     <child link="base_link" />
@@ -275,5 +275,5 @@
   <xacro:include filename="$(find nexus_4wd_mecanum_description)/urdf/nexus_4wd_mecanum.gazebo" />
 <xacro:realsense_d435 sensor_name="d435" parent_link="base_link" rate="10">
-    <origin rpy="0 0 0 " xyz="0.22908 0.09618 0.15"/>
+    <origin rpy="0 0 0 " xyz="0.22908 0.09618 0.05"/>
   </xacro:realsense_d435>
   <xacro:realsense_T265 sensor_name="camera" parent_link="base_link" rate="30.0">

Commit message: simulation_v_3

File: nexus_4wd_mecanum_simulator/nexus_4wd_mecanum_description/urdf/nexus_4wd_mecanum.xacro (robot description, xacro)
@@ -12,5 +12,5 @@
   <link name="base_footprint"></link>
   <joint name="base_link_joint" type="fixed">
-    <origin xyz="1 -0.18 0.05" rpy="0 0 0" />
+    <origin xyz="0 0 0.05" rpy="0 0 0" />
     <parent link="base_footprint"/>
     <child link="base_link" />
@@ -275,8 +275,8 @@
   <xacro:include filename="$(find nexus_4wd_mecanum_description)/urdf/nexus_4wd_mecanum.gazebo" />
 <xacro:realsense_d435 sensor_name="d435" parent_link="base_link" rate="10">
-    <origin rpy="0 0 0 " xyz="0.22908 0.09618 0.05"/>
+    <origin rpy="0 0 0 " xyz="0.22908 0.09618 0.25"/>
   </xacro:realsense_d435>
   <xacro:realsense_T265 sensor_name="camera" parent_link="base_link" rate="30.0">
-    <origin rpy="0 0 0" xyz="0.22908 0.09618 0.30"/>
+    <origin rpy="0 0 0" xyz="0.22908 0.09618 0.1"/>
   </xacro:realsense_T265>
 </robot>

Commit message: simulation_v_4

File: nexus_4wd_mecanum_simulator/nexus_4wd_mecanum_description/urdf/nexus_4wd_mecanum.xacro (robot description, xacro)
@@ -275,5 +275,5 @@
   <xacro:include filename="$(find nexus_4wd_mecanum_description)/urdf/nexus_4wd_mecanum.gazebo" />
 <xacro:realsense_d435 sensor_name="d435" parent_link="base_link" rate="10">
-    <origin rpy="0 0 0 " xyz="0.22908 0.09618 0.25"/>
+    <origin rpy="0 0 0 " xyz="0.22908 0.09618 0.8"/>
   </xacro:realsense_d435>
   <xacro:realsense_T265 sensor_name="camera" parent_link="base_link" rate="30.0">

Commit message: simulation_v_5

File: nexus_4wd_mecanum_simulator/nexus_4wd_mecanum_description/urdf/nexus_4wd_mecanum.xacro (robot description, xacro)
@@ -275,5 +275,5 @@
   <xacro:include filename="$(find nexus_4wd_mecanum_description)/urdf/nexus_4wd_mecanum.gazebo" />
 <xacro:realsense_d435 sensor_name="d435" parent_link="base_link" rate="10">
-    <origin rpy="0 0 0 " xyz="0.22908 0.09618 0.8"/>
+    <origin rpy="0 0 0 " xyz="0.22908 0.09618 0.20"/>
   </xacro:realsense_d435>
   <xacro:realsense_T265 sensor_name="camera" parent_link="base_link" rate="30.0">

Commit message: ccamera_test_v1

File: nexus_4wd_mecanum_simulator/nexus_4wd_mecanum_description/urdf/nexus_4wd_mecanum.xacro (robot description, xacro)
@@ -275,5 +275,5 @@
   <xacro:include filename="$(find nexus_4wd_mecanum_description)/urdf/nexus_4wd_mecanum.gazebo" />
 <xacro:realsense_d435 sensor_name="d435" parent_link="base_link" rate="10">
-    <origin rpy="0 0 0 " xyz="0.22908 0.09618 0.20"/>
+    <origin rpy="0 0 0 " xyz="0.22908 0.09618 0.262"/>
   </xacro:realsense_d435>
   <xacro:realsense_T265 sensor_name="camera" parent_link="base_link" rate="30.0">
